Commit message: 111

File: ros2_vision_project/ros2_ws/src/rc2026_bringup/urdf/rc2026_robot.urdf.xacro (robot description, xacro)
@@ -5,7 +5,10 @@
        底盘: 八边形框架 + 四轮万向轮
        传感器: D435i 相机 + Mid-360S 激光雷达
-       机械臂: 占位符 link, 待组员开发后替换
+       机械臂: 武器头臂 + KFS臂 (含USB相机和吸盘)
+       ★ 所有安装参数来源: robot_params.yaml
+         由 robot_bringup.launch.py 读取后作为 xacro:arg 传入
+         直接修改 robot_params.yaml 即可，无需手动改此文件 ★
        ============================================================ -->
-  <!-- 底盘参数 (可通过 xacro 参数覆盖) -->
+  <!-- ══════════ 底盘几何参数 ══════════ -->
   <xacro:arg name="chassis_width"   default="0.80003"/>
   <xacro:arg name="chassis_depth"   default="0.70025"/>
@@ -15,15 +18,46 @@
   <xacro:arg name="wheel_base_x"    default="0.27"/>
   <xacro:arg name="wheel_base_y"    default="0.25"/>
-  <!-- 传感器安装位置 -->
-  <xacro:arg name="camera_x" default="0.05"/>
-  <xacro:arg name="camera_y" default="0.0"/>
-  <xacro:arg name="camera_z" default="0.45"/>
-  <xacro:arg name="lidar_x"  default="0.0"/>
-  <xacro:arg name="lidar_y"  default="0.0"/>
-  <xacro:arg name="lidar_z"  default="0.55"/>
-  <!-- 机械臂安装位置 -->
-  <xacro:arg name="arm_x" default="0.0"/>
-  <xacro:arg name="arm_y" default="0.0"/>
-  <xacro:arg name="arm_z" default="0.05"/>
+  <!-- ══════════ D435i 相机安装参数 ══════════ -->
+  <xacro:arg name="camera_x"     default="0.05"/>
+  <xacro:arg name="camera_y"     default="0.0"/>
+  <xacro:arg name="camera_z"     default="0.45"/>
+  <xacro:arg name="camera_roll"  default="0.0"/>
+  <xacro:arg name="camera_pitch" default="0.0"/>
+  <xacro:arg name="camera_yaw"   default="0.0"/>
+  <!-- ══════════ Livox Mid-360S 激光雷达安装参数 ══════════ -->
+  <xacro:arg name="lidar_x"     default="0.0"/>
+  <xacro:arg name="lidar_y"     default="0.0"/>
+  <xacro:arg name="lidar_z"     default="0.55"/>
+  <xacro:arg name="lidar_roll"  default="0.0"/>
+  <xacro:arg name="lidar_pitch" default="0.0"/>
+  <xacro:arg name="lidar_yaw"   default="0.0"/>
+  <!-- ══════════ 武器头机械臂安装参数 ══════════ -->
+  <xacro:arg name="weapon_arm_x"     default="0.05"/>
+  <xacro:arg name="weapon_arm_y"     default="0.15"/>
+  <xacro:arg name="weapon_arm_z"     default="0.30"/>
+  <xacro:arg name="weapon_arm_roll"  default="0.0"/>
+  <xacro:arg name="weapon_arm_pitch" default="0.0"/>
+  <xacro:arg name="weapon_arm_yaw"   default="0.0"/>
+  <!-- ══════════ KFS机械臂底座安装参数 ══════════ -->
+  <xacro:arg name="kfs_arm_x"     default="0.0"/>
+  <xacro:arg name="kfs_arm_y"     default="0.0"/>
+  <xacro:arg name="kfs_arm_z"     default="0.05"/>
+  <xacro:arg name="kfs_arm_roll"  default="0.0"/>
+  <xacro:arg name="kfs_arm_pitch" default="0.0"/>
+  <xacro:arg name="kfs_arm_yaw"   default="0.0"/>
+  <!-- ══════════ KFS机械臂展开末端位置（相对arm_base_link）══════════ -->
+  <xacro:arg name="kfs_deployed_x" default="0.30"/>
+  <xacro:arg name="kfs_deployed_y" default="0.0"/>
+  <xacro:arg name="kfs_deployed_z" default="0.40"/>
+  <!-- ══════════ USB相机安装参数（相对arm_deployed_link，镜头朝下）══════════ -->
+  <xacro:arg name="usb_cam_x"     default="0.0"/>
+  <xacro:arg name="usb_cam_y"     default="0.0"/>
+  <xacro:arg name="usb_cam_z"     default="0.0"/>
+  <xacro:arg name="usb_cam_pitch" default="1.5708"/>
+  <!-- ══════════ 吸盘安装参数（相对arm_deployed_link）══════════ -->
+  <xacro:arg name="suction_x" default="0.03"/>
+  <xacro:arg name="suction_y" default="0.0"/>
+  <xacro:arg name="suction_z" default="-0.02"/>
+  <!-- ══════════ 属性 (xacro:arg 的简写别名) ══════════ -->
   <xacro:property name="cw"  value="$(arg chassis_width)"/>
   <xacro:property name="cd"  value="$(arg chassis_depth)"/>
@@ -33,20 +67,11 @@
   <xacro:property name="wbx" value="$(arg wheel_base_x)"/>
   <xacro:property name="wby" value="$(arg wheel_base_y)"/>
-  <!-- ══════════════ 材质定义 ══════════════ -->
-  <material name="grey">
-    <color rgba="0.6 0.6 0.6 1.0"/>
-  </material>
-  <material name="dark_grey">
-    <color rgba="0.3 0.3 0.3 1.0"/>
-  </material>
-  <material name="red">
-    <color rgba="0.8 0.1 0.1 1.0"/>
-  </material>
-  <material name="blue">
-    <color rgba="0.1 0.1 0.8 1.0"/>
-  </material>
-  <material name="green">
-    <color rgba="0.1 0.6 0.1 1.0"/>
-  </material>
+  <!-- ══════════ 材质定义 ══════════ -->
+  <material name="grey">      <color rgba="0.6 0.6 0.6 1.0"/></material>
+  <material name="dark_grey"> <color rgba="0.3 0.3 0.3 1.0"/></material>
+  <material name="red">       <color rgba="0.8 0.1 0.1 1.0"/></material>
+  <material name="blue">      <color rgba="0.1 0.1 0.8 1.0"/></material>
+  <material name="green">     <color rgba="0.1 0.6 0.1 1.0"/></material>
+  <material name="yellow">    <color rgba="0.9 0.8 0.1 1.0"/></material>
   <!-- ══════════════ base_footprint ══════════════ -->
   <link name="base_footprint"/>
@@ -59,14 +84,10 @@
   <link name="base_link">
     <visual>
-      <geometry>
-        <box size="${cw} ${cd} 0.08"/>
-      </geometry>
+      <geometry><box size="${cw} ${cd} 0.08"/></geometry>
       <origin xyz="0 0 0.04" rpy="0 0 0"/>
       <material name="red"/>
     </visual>
     <collision>
-      <geometry>
-        <box size="${cw} ${cd} 0.08"/>
-      </geometry>
+      <geometry><box size="${cw} ${cd} 0.08"/></geometry>
       <origin xyz="0 0 0.04" rpy="0 0 0"/>
     </collision>
@@ -79,14 +100,10 @@
   <link name="frame_upper">
     <visual>
-      <geometry>
-        <box size="${cw} ${cd} ${ch}"/>
-      </geometry>
+      <geometry><box size="${cw} ${cd} ${ch}"/></geometry>
       <origin xyz="0 0 ${ch/2}" rpy="0 0 0"/>
       <material name="grey"/>
     </visual>
     <collision>
-      <geometry>
-        <box size="${cw} ${cd} ${ch}"/>
-      </geometry>
+      <geometry><box size="${cw} ${cd} ${ch}"/></geometry>
       <origin xyz="0 0 ${ch/2}" rpy="0 0 0"/>
     </collision>
@@ -106,14 +123,10 @@
     <link name="${name}_link">
       <visual>
-        <geometry>
-          <cylinder radius="${wr}" length="${ww}"/>
-        </geometry>
+        <geometry><cylinder radius="${wr}" length="${ww}"/></geometry>
         <origin xyz="0 0 0" rpy="${pi/2} 0 0"/>
         <material name="dark_grey"/>
       </visual>
       <collision>
-        <geometry>
-          <cylinder radius="${wr}" length="${ww}"/>
-        </geometry>
+        <geometry><cylinder radius="${wr}" length="${ww}"/></geometry>
         <origin xyz="0 0 0" rpy="${pi/2} 0 0"/>
       </collision>
@@ -131,21 +144,16 @@
     </joint>
   </xacro:macro>
-  <!-- 四个万向轮 -->
   <xacro:omni_wheel name="wheel_fl" x="${wbx}"  y="${wby}"/>
   <xacro:omni_wheel name="wheel_fr" x="${wbx}"  y="${-wby}"/>
   <xacro:omni_wheel name="wheel_rl" x="${-wbx}" y="${wby}"/>
   <xacro:omni_wheel name="wheel_rr" x="${-wbx}" y="${-wby}"/>
-  <!-- ══════════════ 相机 (Intel RealSense D435i) ══════════════ -->
+  <!-- ══════════════ D435i 主视觉相机 ══════════════ -->
   <link name="camera_link">
     <visual>
-      <geometry>
-        <box size="0.025 0.09 0.025"/>
-      </geometry>
+      <geometry><box size="0.025 0.09 0.025"/></geometry>
       <material name="grey"/>
     </visual>
     <collision>
-      <geometry>
-        <box size="0.025 0.09 0.025"/>
-      </geometry>
+      <geometry><box size="0.025 0.09 0.025"/></geometry>
     </collision>
     <inertial>
@@ -158,5 +166,5 @@
     <child link="camera_link"/>
     <origin xyz="$(arg camera_x) $(arg camera_y) $(arg camera_z)"
-            rpy="0 0 0"/>
+            rpy="$(arg camera_roll) $(arg camera_pitch) $(arg camera_yaw)"/>
   </joint>
   <!-- D435i 光学坐标系 (Z前 X右 Y下) -->
@@ -167,16 +175,12 @@
     <origin xyz="0 0 0" rpy="${-pi/2} 0 ${-pi/2}"/>
   </joint>
-  <!-- ══════════════ 激光雷达 (Livox Mid-360S) ══════════════ -->
+  <!-- ══════════════ Livox Mid-360S 激光雷达 ══════════════ -->
   <link name="lidar_link">
     <visual>
-      <geometry>
-        <cylinder radius="0.05" length="0.06"/>
-      </geometry>
+      <geometry><cylinder radius="0.05" length="0.06"/></geometry>
       <material name="blue"/>
     </visual>
     <collision>
-      <geometry>
-        <cylinder radius="0.05" length="0.06"/>
-      </geometry>
+      <geometry><cylinder radius="0.05" length="0.06"/></geometry>
     </collision>
     <inertial>
@@ -189,22 +193,16 @@
     <child link="lidar_link"/>
     <origin xyz="$(arg lidar_x) $(arg lidar_y) $(arg lidar_z)"
-            rpy="0 0 0"/>
-  </joint>
-  <!-- ══════════════ 武器头机械臂底座 (占位, 位置待定, 需现场测量标定) ══════════════ -->
-  <!-- 用于夹取武器端头, 拾取/释放指令由 ActionGroupCmd id=1/2 发送,
-       下位机自动控制对应机械臂, 上位机无需区分两臂。
-       安装位置不会远离 D435i 相机(camera_link), 下方 xyz 为临时占位,
-       确定安装点后用卷尺测量相对 base_link 的实际偏移并替换。 -->
+            rpy="$(arg lidar_roll) $(arg lidar_pitch) $(arg lidar_yaw)"/>
+  </joint>
+  <!-- ══════════════ 武器头机械臂底座 ══════════════ -->
+  <!-- 功能: 拾取/释放武器端头 (ActionGroupCmd id=1/2)
+       安装位置: ★ 待现场测量后通过 robot_params.yaml 修改 ★ -->
   <link name="weapon_arm_base_link">
     <visual>
-      <geometry>
-        <cylinder radius="0.03" length="0.02"/>
-      </geometry>
-      <material name="blue"/>
-    </visual>
-    <collision>
-      <geometry>
-        <cylinder radius="0.03" length="0.02"/>
-      </geometry>
+      <geometry><cylinder radius="0.03" length="0.02"/></geometry>
+      <material name="yellow"/>
+    </visual>
+    <collision>
+      <geometry><cylinder radius="0.03" length="0.02"/></geometry>
     </collision>
     <inertial>
@@ -216,19 +214,17 @@
     <parent link="base_link"/>
     <child link="weapon_arm_base_link"/>
-    <!-- TODO: 现场测量后替换 xyz，当前为占位值 (靠近相机前方) -->
-    <origin xyz="0.05 0.15 0.30" rpy="0 0 0"/>
-  </joint>
-  <!-- ══════════════ KFS机械臂底座 (占位符, 待组员替换) ══════════════ -->
+    <origin xyz="$(arg weapon_arm_x) $(arg weapon_arm_y) $(arg weapon_arm_z)"
+            rpy="$(arg weapon_arm_roll) $(arg weapon_arm_pitch) $(arg weapon_arm_yaw)"/>
+  </joint>
+  <!-- ══════════════ KFS机械臂底座 ══════════════ -->
+  <!-- 功能: 梅林区精对齐 + 吸盘拾取KFS
+       安装位置: ★ 待现场测量后通过 robot_params.yaml 修改 ★ -->
   <link name="arm_base_link">
     <visual>
-      <geometry>
-        <cylinder radius="0.03" length="0.02"/>
-      </geometry>
+      <geometry><cylinder radius="0.03" length="0.02"/></geometry>
       <material name="green"/>
     </visual>
     <collision>
-      <geometry>
-        <cylinder radius="0.03" length="0.02"/>
-      </geometry>
+      <geometry><cylinder radius="0.03" length="0.02"/></geometry>
     </collision>
     <inertial>
@@ -240,31 +236,26 @@
     <parent link="base_link"/>
     <child link="arm_base_link"/>
-    <origin xyz="$(arg arm_x) $(arg arm_y) $(arg arm_z)"
-            rpy="0 0 0"/>
-  </joint>
-  <!-- ══════════════ 机械臂展开姿态 (精对齐用, 占位几何, 需现场标定) ══════════════ -->
-  <!-- 代表机械臂完全抬升+前伸+末端旋转朝下后(精对齐动作组完成姿态),
-       末端横杆中心相对 arm_base_link 的固定位姿。
-       现实现为固定坐标系(单一展开姿态), 不建模抬升/前伸的连续关节,
-       因为精对齐阶段不调整机械臂本身位姿, 误差直接转换为底盘 vx/vy。
-       下方 xyz 数值为占位估测, 需结合实物测量校正。 -->
+    <origin xyz="$(arg kfs_arm_x) $(arg kfs_arm_y) $(arg kfs_arm_z)"
+            rpy="$(arg kfs_arm_roll) $(arg kfs_arm_pitch) $(arg kfs_arm_yaw)"/>
+  </joint>
+  <!-- ══════════════ KFS机械臂展开末端 ══════════════ -->
+  <!-- 代表机械臂完全抬升+前伸后末端中心的固定位姿
+       精对齐阶段不调整机械臂关节，误差转换为底盘 vx/vy
+       ★ 待实测机械臂展开尺寸后通过 robot_params.yaml 修改 ★ -->
   <link name="arm_deployed_link"/>
   <joint name="arm_deployed_joint" type="fixed">
     <parent link="arm_base_link"/>
     <child link="arm_deployed_link"/>
-    <origin xyz="0.30 0 0.40" rpy="0 0 0"/>
-  </joint>
-  <!-- ══════════════ USB 相机 (末端横杆, 精对齐用, 镜头朝下) ══════════════ -->
+    <origin xyz="$(arg kfs_deployed_x) $(arg kfs_deployed_y) $(arg kfs_deployed_z)"
+            rpy="0 0 0"/>
+  </joint>
+  <!-- ══════════════ USB相机 (KFS臂末端, 精对齐用, 镜头朝下) ══════════════ -->
   <link name="usb_camera_link">
     <visual>
-      <geometry>
-        <box size="0.03 0.03 0.03"/>
-      </geometry>
+      <geometry><box size="0.03 0.03 0.03"/></geometry>
       <material name="dark_grey"/>
     </visual>
     <collision>
-      <geometry>
-        <box size="0.03 0.03 0.03"/>
-      </geometry>
+      <geometry><box size="0.03 0.03 0.03"/></geometry>
     </collision>
     <inertial>
@@ -276,8 +267,9 @@
     <parent link="arm_deployed_link"/>
     <child link="usb_camera_link"/>
-    <!-- 镜头朝下: 绕Y轴+90°使 camera_link 的 X(前) 轴指向 -Z(地面) -->
-    <origin xyz="0 0 0" rpy="0 ${pi/2} 0"/>
-  </joint>
-  <!-- USB 相机光学坐标系 (Z指向镜头朝向/地面, X右 Y下), 供图像处理使用 -->
+    <!-- pitch=π/2 使相机X轴（前方）朝向-Z（地面），实现镜头朝下 -->
+    <origin xyz="$(arg usb_cam_x) $(arg usb_cam_y) $(arg usb_cam_z)"
+            rpy="0 $(arg usb_cam_pitch) 0"/>
+  </joint>
+  <!-- USB相机光学坐标系 (Z指向镜头朝向/地面, X右 Y下) -->
   <link name="usb_camera_optical_frame"/>
   <joint name="usb_camera_optical_joint" type="fixed">
@@ -286,16 +278,13 @@
     <origin xyz="0 0 0" rpy="${-pi/2} 0 ${-pi/2}"/>
   </joint>
-  <!-- ══════════════ 吸盘 (末端横杆, 与USB相机存在小偏移, 需现场标定) ══════════════ -->
+  <!-- ══════════════ 吸盘 (KFS臂末端, 与USB相机存在小偏移) ══════════════ -->
+  <!-- ★ 待现场测量后通过 robot_params.yaml 修改 suction_x/y/z ★ -->
   <link name="suction_link">
     <visual>
-      <geometry>
-        <cylinder radius="0.025" length="0.02"/>
-      </geometry>
+      <geometry><cylinder radius="0.025" length="0.02"/></geometry>
       <material name="green"/>
     </visual>
     <collision>
-      <geometry>
-        <cylinder radius="0.025" length="0.02"/>
-      </geometry>
+      <geometry><cylinder radius="0.025" length="0.02"/></geometry>
     </collision>
     <inertial>
@@ -307,5 +296,5 @@
     <parent link="arm_deployed_link"/>
     <child link="suction_link"/>
-    <origin xyz="0.03 0 -0.02" rpy="0 0 0"/>
+    <origin xyz="$(arg suction_x) $(arg suction_y) $(arg suction_z)" rpy="0 0 0"/>
   </joint>
 </robot>
